File: RaspberryPIFullStackHAT/RaspberryPIFullStackHAT/RaspberryPIFullStackHAT.sch (KiCad schematic (older format))
At the start: 7 parts, among them J1 Raspberry_Pi_2_3, SW1 SW_DPST, U1 DHT22

Commit message: work on raspberry pi hat
Parts:
- added D2: LED, LED_SMD:LED_0805_2012Metric, symbol Device:LED
- added R4: R, Resistor_SMD:R_0805_2012Metric, symbol Device:R
Connections:
- net +3V3: now reaches J1.1 (3V3)
- net +3V3: now also R2.1, SW1.1, SW1.3, U1.1 (VCC), R4.2
- net DHT22_input: now reaches J1.11 (GPIO17)
- net DHT22_input: now also R2.2, U1.2 (IO)
- net GND: now reaches J1.6 (GND)
- net GND: now also D1.1 (K), J1.9 (GND), R1.1, U1.4 (GND), D2.1 (K)
- net led_output: now reaches J1.7 (GCLK0/GPIO4)
- net led_output: now also R3.2
- net button_input: now reaches J1.8 (GPIO14/TXD)
- net button_input: now also R1.2, SW1.2, SW1.4
- net at R3.1: now also D1.2 (A)
- new net: D2.2 (A), R4.1
- no-connect marks 0 -> 34
Other:
- note added: "N1 - momentary button"
- note added: "N2 - sensor DHT22"
- note added: "N3 - Raspberry Pi"
- note added: "N4 - indicator led"
- note added: "N5 - power indicator led"
- note added: "POWER FLAGS"
- moved on the sheet: D1, J1, R1, R2, R3, SW1, U1

Commit message: no message
Parts:
- J1: footprint Connector_PinSocket_2.54mm:PinSocket_2x08_P2.54mm_Vertical -> Connector_PinHeader_2.54mm:PinHeader_2x08_P2.54mm_Vertical
- U1: footprint Connector_PinHeader_2.54mm:PinHeader_1x03_P2.54mm_Vertical -> Connector_PinHeader_2.54mm:PinHeader_1x04_P2.54mm_Vertical
Changed lines of the file:
@@
 F 0 "U1" H 3356 4146 50  0000 R CNN
 F 1 "DHT22" H 3356 4055 50  0000 R CNN
-F 2 "Connector_PinHeader_2.54mm:PinHeader_1x03_P2.54mm_Vertical" H 3600 3700 50  0001 C CNN
+F 2 "Connector_PinHeader_2.54mm:PinHeader_1x04_P2.54mm_Vertical" H 3600 3700 50  0001 C CNN
 F 3 "http://akizukidenshi.com/download/ds/aosong/DHT11.pdf" H 3750 4350 50  0001 C CNN
 	1    3600 4100
@@
 F 0 "J1" H 8150 5131 50  0000 C CNN
 F 1 "Raspberry_Pi_2_3" H 8150 5040 50  0000 C CNN
-F 2 "Connector_PinSocket_2.54mm:PinSocket_2x08_P2.54mm_Vertical" H 8150 3650 50  0001 C CNN
+F 2 "Connector_PinHeader_2.54mm:PinHeader_2x08_P2.54mm_Vertical" H 8150 3650 50  0001 C CNN
 F 3 "https://www.raspberrypi.org/documentation/hardware/raspberrypi/schematics/rpi_SCH_3bplus_1p0_reduced.pdf" H 8150 3650 50  0001 C CNN
 	1    8150 3650
